Commit message: update s500 urdf and yaml files, add s500_simple with fixed rotor

File: eagle_mpc_yaml/s500_robot/s500_quadrotor/urdf/s500_simple.urdf (robot description, URDF)
Before this commit: robot s500_quadrotor, 5 links, 4 joints
Joints:
- joint rotor_joint_1: type continuous -> fixed
- joint rotor_joint_2: type continuous -> fixed
- joint rotor_joint_3: type continuous -> fixed
- joint rotor_joint_4: type continuous -> fixed
