Commit message: update s500 trajectory and mpc config file

File: eagle_mpc_yaml/s500_robot/s500_quadrotor/urdf/s500_quadrotor.urdf (robot description, URDF)
Before this commit: robot s500_quadrotor, 5 links, 4 joints
Links:
- removed link s500_base_link
- added link base_link, mass 1.772; collision mesh filename=package://s500_quadrotor/meshes/base_link.STL; visual mesh filename=package://s500_quadrotor/meshes/base_link.STL

File: eagle_mpc_yaml/s500_robot/s500_quadrotor/urdf/s500_simple.urdf (robot description, URDF)
Before this commit: robot s500_quadrotor, 5 links, 4 joints
Links:
- removed link s500_base_link
- added link base_link, mass 1.772; collision mesh filename=package://s500_quadrotor/meshes/base_link.STL; visual mesh filename=package://s500_quadrotor/meshes/base_link.STL

Commit message: update s500 model with iris prop

File: eagle_mpc_yaml/s500_robot/s500_quadrotor/urdf/s500_quadrotor.urdf (robot description, URDF)
Before this commit: robot s500_quadrotor, 5 links, 4 joints
Links:
- link rotor_1: geometry collision mesh filename=package://s500_quadrotor/meshes/rotor_1.STL; visual mesh filename=package://s500_quadrotor/meshes/iris_prop_ccw.dae
- link rotor_2: geometry collision mesh filename=package://s500_quadrotor/meshes/rotor_2.STL; visual mesh filename=package://s500_quadrotor/meshes/iris_prop_ccw.dae
- link rotor_3: geometry collision mesh filename=package://s500_quadrotor/meshes/rotor_3.STL; visual mesh filename=package://s500_quadrotor/meshes/iris_prop_cw.dae
- link rotor_4: geometry collision mesh filename=package://s500_quadrotor/meshes/rotor_4.STL; visual mesh filename=package://s500_quadrotor/meshes/iris_prop_cw.dae

Commit message: updated s500 robot urdf

File: eagle_mpc_yaml/s500_robot/s500_quadrotor/urdf/s500_quadrotor.urdf (robot description, URDF)
Before this commit: robot s500_quadrotor, 5 links, 4 joints
Links:
- link base_link: geometry collision mesh filename=package://eagle_mpc_yaml/s500_robot/s500_quadrotor/meshes/b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; visual mesh filename=package://eagle_mpc_yaml/s500_robot/s500_quadrotor/meshes/b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
- link rotor_1: geometry collision mesh filename=package://eagle_mpc_yaml/s500_robot/s500_quadrotor/meshes/r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; visual mesh filename=package://eagle_mpc_yaml/s500_robot/s500_quadrotor/meshes/i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
- link rotor_2: geometry collision mesh filename=package://eagle_mpc_yaml/s500_robot/s500_quadrotor/meshes/r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; visual mesh filename=package://eagle_mpc_yaml/s500_robot/s500_quadrotor/meshes/i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
- link rotor_3: geometry collision mesh filename=package://eagle_mpc_yaml/s500_robot/s500_quadrotor/meshes/r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; visual mesh filename=package://eagle_mpc_yaml/s500_robot/s500_quadrotor/meshes/i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
- link rotor_4: geometry collision mesh filename=package://eagle_mpc_yaml/s500_robot/s500_quadrotor/meshes/r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; visual mesh filename=package://eagle_mpc_yaml/s500_robot/s500_quadrotor/meshes/i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

File: eagle_mpc_yaml/s500_robot/s500_quadrotor/urdf/s500_simple.urdf (robot description, URDF)
Before this commit: robot s500_quadrotor, 5 links, 4 joints
Links:
- link base_link: geometry collision mesh filename=package://eagle_mpc_yaml/s500_robot/s500_quadrotor/meshes/b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; visual mesh filename=package://eagle_mpc_yaml/s500_robot/s500_quadrotor/meshes/b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
- link rotor_1: geometry collision mesh filename=package://eagle_mpc_yaml/s500_robot/s500_quadrotor/meshes/r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; visual mesh filename=package://eagle_mpc_yaml/s500_robot/s500_quadrotor/meshes/r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
- link rotor_2: geometry collision mesh filename=package://eagle_mpc_yaml/s500_robot/s500_quadrotor/meshes/r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; visual mesh filename=package://eagle_mpc_yaml/s500_robot/s500_quadrotor/meshes/r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
- link rotor_3: geometry collision mesh filename=package://eagle_mpc_yaml/s500_robot/s500_quadrotor/meshes/r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; visual mesh filename=package://eagle_mpc_yaml/s500_robot/s500_quadrotor/meshes/r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
- link rotor_4: geometry collision mesh filename=package://eagle_mpc_yaml/s500_robot/s500_quadrotor/meshes/r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; visual mesh filename=package://eagle_mpc_yaml/s500_robot/s500_quadrotor/meshes/r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

File: eagle_mpc_yaml/s500_robot/s500_uam/urdf/s500_uam.urdf (robot description, URDF)
Before this commit: robot s500_uam, 9 links, 8 joints
Links:
- link base_link: geometry collision mesh filename=package://eagle_mpc_yaml/s500_robot/s500_quadrotor/meshes/b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; visual mesh filename=package://eagle_mpc_yaml/s500_robot/s500_quadrotor/meshes/b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
- link link_1: geometry collision mesh filename=package://eagle_mpc_yaml/s500_robot/s500_uam/meshes/link_1.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; visual mesh filename=package://eagle_mpc_yaml/s500_robot/s500_uam/meshes/link_1.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
- link link_2: geometry collision mesh filename=package://eagle_mpc_yaml/s500_robot/s500_uam/meshes/link_2.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; visual mesh filename=package://eagle_mpc_yaml/s500_robot/s500_uam/meshes/link_2.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
- link link_3: geometry collision mesh filename=package://eagle_mpc_yaml/s500_robot/s500_uam/meshes/link_3.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; visual mesh filename=package://eagle_mpc_yaml/s500_robot/s500_uam/meshes/link_3.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
- link link_4: geometry collision mesh filename=package://eagle_mpc_yaml/s500_robot/s500_uam/meshes/link_4.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; visual mesh filename=package://eagle_mpc_yaml/s500_robot/s500_uam/meshes/link_4.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
- link rotor_1: geometry collision mesh filename=package://eagle_mpc_yaml/s500_robot/s500_quadrotor/meshes/r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; visual mesh filename=package://eagle_mpc_yaml/s500_robot/s500_quadrotor/meshes/i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
- link rotor_2: geometry collision mesh filename=package://eagle_mpc_yaml/s500_robot/s500_quadrotor/meshes/r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; visual mesh filename=package://eagle_mpc_yaml/s500_robot/s500_quadrotor/meshes/i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
- link rotor_3: geometry collision mesh filename=package://eagle_mpc_yaml/s500_robot/s500_quadrotor/meshes/r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; visual mesh filename=package://eagle_mpc_yaml/s500_robot/s500_quadrotor/meshes/i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
- link rotor_4: geometry collision mesh filename=package://eagle_mpc_yaml/s500_robot/s500_quadrotor/meshes/r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; visual mesh filename=package://eagle_mpc_yaml/s500_robot/s500_quadrotor/meshes/i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

Commit message: update s500 quadrotor urdf

File: eagle_mpc_yaml/s500_robot/s500_quadrotor/urdf/s500_quadrotor.urdf (robot description, URDF)
Before this commit: robot s500_quadrotor, 5 links, 4 joints
Links:
- link rotor_1: geometry collision mesh filename=package://eagle_mpc_yaml/s500_robot/s500_quadrotor/meshes/i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; visual mesh filename=package://eagle_mpc_yaml/s500_robot/s500_quadrotor/meshes/i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
- link rotor_2: geometry collision mesh filename=package://eagle_mpc_yaml/s500_robot/s500_quadrotor/meshes/i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; visual mesh filename=package://eagle_mpc_yaml/s500_robot/s500_quadrotor/meshes/i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
- link rotor_3: geometry collision mesh filename=package://eagle_mpc_yaml/s500_robot/s500_quadrotor/meshes/i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; visual mesh filename=package://eagle_mpc_yaml/s500_robot/s500_quadrotor/meshes/i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
- link rotor_4: geometry collision mesh filename=package://eagle_mpc_yaml/s500_robot/s500_quadrotor/meshes/i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; visual mesh filename=package://eagle_mpc_yaml/s500_robot/s500_quadrotor/meshes/i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

File: eagle_mpc_yaml/s500_robot/s500_quadrotor/urdf/s500_simple.urdf (robot description, URDF)
Before this commit: robot s500_quadrotor, 5 links, 4 joints
Links:
- link rotor_1: geometry collision mesh filename=package://eagle_mpc_yaml/s500_robot/s500_quadrotor/meshes/i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; visual mesh filename=package://eagle_mpc_yaml/s500_robot/s500_quadrotor/meshes/i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
- link rotor_2: geometry collision mesh filename=package://eagle_mpc_yaml/s500_robot/s500_quadrotor/meshes/i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; visual mesh filename=package://eagle_mpc_yaml/s500_robot/s500_quadrotor/meshes/i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
- link rotor_3: geometry collision mesh filename=package://eagle_mpc_yaml/s500_robot/s500_quadrotor/meshes/i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; visual mesh filename=package://eagle_mpc_yaml/s500_robot/s500_quadrotor/meshes/i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
- link rotor_4: geometry collision mesh filename=package://eagle_mpc_yaml/s500_robot/s500_quadrotor/meshes/i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; visual mesh filename=package://eagle_mpc_yaml/s500_robot/s500_quadrotor/meshes/i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
