Commit message: update s500_uam config

File: eagle_mpc_yaml/s500_robot/s500_uam/urdf/s500_uam.urdf (robot description, URDF)
Before this commit: robot s500_uam, 5 links, 4 joints
Links:
- added link rotor_1, mass 0.010198; collision mesh filename=package://s500_quadrotor/meshes/rotor_1.STL; visual mesh filename=package://s500_quadrotor/meshes/iris_prop_ccw.dae
- added link rotor_2, mass 0.010198; collision mesh filename=package://s500_quadrotor/meshes/rotor_2.STL; visual mesh filename=package://s500_quadrotor/meshes/iris_prop_ccw.dae
- added link rotor_3, mass 0.010198; collision mesh filename=package://s500_quadrotor/meshes/rotor_3.STL; visual mesh filename=package://s500_quadrotor/meshes/iris_prop_cw.dae
- added link rotor_4, mass 0.010198; collision mesh filename=package://s500_quadrotor/meshes/rotor_4.STL; visual mesh filename=package://s500_quadrotor/meshes/iris_prop_cw.dae
- link base_link: mass 1.5 -> 1.772; geometry collision mesh filename=package://s500_quadrotor/meshes/base_link.STL; visual mesh filename=package://s500_quadrotor/meshes/base_link.STL
Joints:
- added joint rotor_joint_1: type continuous, parent base_link, child rotor_1, origin xyz=0.171 0.171 0.045 rpy=0 0 0, axis 0 1 0
- added joint rotor_joint_2: type continuous, parent base_link, child rotor_2, origin xyz=-0.171 0.171 0.045 rpy=0 0 0, axis 0 1 0
- added joint rotor_joint_3: type continuous, parent base_link, child rotor_3, origin xyz=-0.171 -0.171 0.045 rpy=0 0 0, axis 0 1 0
- added joint rotor_joint_4: type continuous, parent base_link, child rotor_4, origin xyz=0.1701 -0.1701 0.0603 rpy=0 0 0, axis 0 1 0
- joint joint_1: origin xyz=0.0007 0 -0.07275 rpy=0 0 0 -> xyz=0.0007 0 -0.07275 rpy=0 -1 0
- joint joint_2: origin xyz=0 0 -0.09925 rpy=0 0.2936 0 -> xyz=0 0 -0.09925 rpy=0 -0.6 0

File: eagle_mpc_yaml/s500_robot/s500_uam/urdf/s500_uam_simple.urdf (robot description, URDF)
Before this commit: robot s500_uam, 9 links, 8 joints
Links:
- link base_link: geometry collision mesh filename=package://example-robot-data/robots/s500_description/meshes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; visual mesh filename=package://example-robot-data/robots/s500_description/meshes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
- link link_1: geometry collision mesh filename=package://example-robot-data/robots/s500_description/meshes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; visual mesh filename=package://example-robot-data/robots/s500_description/meshes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
- link link_2: geometry collision mesh filename=package://example-robot-data/robots/s500_description/meshes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; visual mesh filename=package://example-robot-data/robots/s500_description/meshes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
- link link_3: geometry collision mesh filename=package://example-robot-data/robots/s500_description/meshes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; visual mesh filename=package://example-robot-data/robots/s500_description/meshes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
- link link_4: geometry collision mesh filename=package://example-robot-data/robots/s500_description/meshes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; visual mesh filename=package://example-robot-data/robots/s500_description/meshes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
- link rotor_1: geometry collision mesh filename=package://example-robot-data/robots/s500_description/meshes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; visual mesh filename=package://example-robot-data/robots/s500_description/meshes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
- link rotor_2: geometry collision mesh filename=package://example-robot-data/robots/s500_description/meshes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; visual mesh filename=package://example-robot-data/robots/s500_description/meshes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
- link rotor_3: geometry collision mesh filename=package://example-robot-data/robots/s500_description/meshes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; visual mesh filename=package://example-robot-data/robots/s500_description/meshes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
- link rotor_4: geometry collision mesh filename=package://example-robot-data/robots/s500_description/meshes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; visual mesh filename=package://example-robot-data/robots/s500_description/meshes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
Joints:
- joint joint_1: limit (none) -> lower=-1.5 upper=1.5 effort=1 velocity=3; origin xyz=0.0007 0 -0.07275 rpy=0 0 0 -> xyz=0.0007 0 -0.07275 rpy=0 -1 0; type continuous -> revolute
- joint joint_2: limit (none) -> lower=-1.5 upper=1.5 effort=1 velocity=3; origin xyz=0 0 -0.09925 rpy=0 0.2936 0 -> xyz=0 0 -0.09925 rpy=0 -0.6 0; type continuous -> revolute
- joint joint_3: type continuous -> fixed
- joint joint_4: type continuous -> fixed
- joint rotor_joint_1: origin xyz=0.171 0.171 0.045 rpy=0 0 0 -> xyz=0.171 0.171 0.07 rpy=0 0 0
- joint rotor_joint_2: origin xyz=-0.171 0.171 0.045 rpy=0 0 0 -> xyz=-0.171 0.171 0.07 rpy=0 0 0
- joint rotor_joint_3: origin xyz=-0.171 -0.171 0.045 rpy=0 0 0 -> xyz=-0.171 -0.171 0.07 rpy=0 0 0
- joint rotor_joint_4: origin xyz=0.1701 -0.1701 0.0603 rpy=0 0 0 -> xyz=0.1701 -0.1701 0.07 rpy=0 0 0
